File: ZigBeeHA/main.sch (EAGLE design)
At the start: 12 parts, among them IC1 REG1117

Commit message: parts updated
parts updated
Parts:
- removed C4: 10uF, resistor:CPOL-US140CLH-0810
- added C5: 10uF, rcl:C-USC1206
- C1, C2, C3: device resistor:CPOL-US140CLH-0810 -> rcl:CPOL-USSANYO_SMD_A5
- R1: device rcl:R-US_0204/7 -> rcl:R-US_M1206
Connections:
- removed net +3V3: C1.+, C3.+, IC1.VOUT, R1.2, SV1.12, SV2.1
- new net VCC: C1.+, C3.+, IC1.VOUT, PAD3.P, R1.2, SV1.12, SV2.1
- net +5V: no longer PAD3.P
- net /RESET: now also C5.1; no longer C4.+
- net GND: now also C5.2; no longer C4.-
Other:
- moved on the sheet: C1, C3, R1
Changed lines of the file:
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@@
 <parts>
 <part name="IC1" library="burr-brown" deviceset="REG1117" device=""/>
-<part name="C2" library="resistor" deviceset="CPOL-US" device="140CLH-0810" value="10uF"/>
-<part name="C4" library="resistor" deviceset="CPOL-US" device="140CLH-0810" value="10uF"/>
-<part name="C3" library="resistor" deviceset="CPOL-US" device="140CLH-0810" value="4.7uF"/>
+<part name="C2" library="rcl" deviceset="CPOL-US" device="SANYO_SMD_A5" value="10uF"/>
+<part name="C3" library="rcl" deviceset="CPOL-US" device="SANYO_SMD_A5" value="4.7uF"/>
 <part name="P+3" library="supply1" deviceset="+5V" device=""/>
 <part name="SUPPLY6" library="supply2" deviceset="GND" device=""/>
 <part name="SUPPLY7" library="supply2" deviceset="GND" device=""/>
-<part name="+3V2" library="supply1" deviceset="+3V3" device=""/>
 <part name="SUPPLY8" library="supply2" deviceset="GND" device=""/>
 <part name="SUPPLY9" library="supply2" deviceset="GND" device=""/>
-<part name="R1" library="rcl" deviceset="R-US_" device="0204/7" value="10K"/>
+<part name="R1" library="rcl" deviceset="R-US_" device="M1206" value="10K"/>
 <part name="P+4" library="supply1" deviceset="+5V" device=""/>
 <part name="SUPPLY10" library="supply2" deviceset="GND" device=""/>
 <part name="PAD1" library="wirepad" deviceset="2,54/0,8" device="" value="+5V"/>
 <part name="PAD2" library="wirepad" deviceset="2,54/0,8" device="" value="GND"/>
-<part name="P+1" library="supply1" deviceset="+5V" device="" value="+3V3"/>
 <part name="PAD3" library="wirepad" deviceset="2,54/0,8" device="" value="+3.3V"/>
 <part name="SV1" library="con-lstb" deviceset="MA13-1" device=""/>
@@
 <part name="SUPPLY1" library="supply2" deviceset="GND" device=""/>
 <part name="SUPPLY2" library="supply2" deviceset="GND" device=""/>
-<part name="+3V1" library="supply1" deviceset="+3V3" device=""/>
-<part name="C1" library="resistor" deviceset="CPOL-US" device="140CLH-0810" value="4.7uF"/>
+<part name="C1" library="rcl" deviceset="CPOL-US" device="SANYO_SMD_A5" value="4.7uF"/>
 <part name="SUPPLY3" library="supply2" deviceset="GND" device=""/>
-<part name="+3V3" library="supply1" deviceset="+3V3" device=""/>
+<part name="SUPPLY4" library="supply2" deviceset="VCC" device="" value="+3.3V"/>
+<part name="SUPPLY13" library="supply2" deviceset="VCC" device="" value="+3.3V"/>
+<part name="SUPPLY14" library="supply2" deviceset="VCC" device="" value="+3.3V"/>
+<part name="SUPPLY15" library="supply2" deviceset="VCC" device="" value="+3.3V"/>
+<part name="C5" library="rcl" deviceset="C-US" device="C1206" value="10uF"/>
 </parts>
 <sheets>
@@
 <instance part="IC1" gate="G$1" x="81.28" y="218.44"/>
 <instance part="C2" gate="G$1" x="60.96" y="213.36"/>
-<instance part="C4" gate="G$1" x="116.84" y="213.36"/>
-<instance part="C3" gate="G$1" x="99.06" y="213.36"/>
+<instance part="C3" gate="G$1" x="96.52" y="213.36"/>
 <instance part="P+3" gate="1" x="60.96" y="228.6"/>
 <instance part="SUPPLY6" gate="GND" x="60.96" y="200.66"/>
-<instance part="SUPPLY7" gate="GND" x="99.06" y="200.66"/>
-<instance part="+3V2" gate="G$1" x="99.06" y="228.6"/>
+<instance part="SUPPLY7" gate="GND" x="96.52" y="200.66"/>
 <instance part="SUPPLY8" gate="GND" x="81.28" y="200.66"/>
-<instance part="SUPPLY9" gate="GND" x="116.84" y="200.66"/>
-<instance part="R1" gate="G$1" x="109.22" y="218.44" rot="R180"/>
+<instance part="SUPPLY9" gate="GND" x="111.76" y="200.66"/>
+<instance part="R1" gate="G$1" x="104.14" y="218.44" rot="R180"/>
 <instance part="P+4" gate="1" x="43.18" y="228.6"/>
 <instance part="SUPPLY10" gate="GND" x="43.18" y="200.66" smashed="yes">
@@
 <attribute name="VALUE" x="39.878" y="209.423" size="1.778" layer="96" rot="R270"/>
 </instance>
-<instance part="P+1" gate="1" x="160.02" y="228.6"/>
 <instance part="PAD3" gate="P" x="160.02" y="218.44" smashed="yes" rot="R90">
 <attribute name="NAME" x="163.2458" y="217.297" size="1.778" layer="95" rot="R90"/>
@@
 <instance part="SUPPLY1" gate="GND" x="58.42" y="139.7"/>
 <instance part="SUPPLY2" gate="GND" x="109.22" y="139.7"/>
-<instance part="+3V1" gate="G$1" x="50.8" y="154.94"/>
-<instance part="C1" gate="G$1" x="50.8" y="144.78"/>
-<instance part="SUPPLY3" gate="GND" x="50.8" y="134.62"/>
-<instance part="+3V3" gate="G$1" x="71.12" y="144.78"/>
+<instance part="C1" gate="G$1" x="50.8" y="142.24"/>
+<instance part="SUPPLY3" gate="GND" x="50.8" y="132.08"/>
+<instance part="SUPPLY4" gate="G$1" x="96.52" y="228.6"/>
+<instance part="SUPPLY13" gate="G$1" x="160.02" y="228.6"/>
+<instance part="SUPPLY14" gate="G$1" x="50.8" y="149.86"/>
+<instance part="SUPPLY15" gate="G$1" x="71.12" y="142.24"/>
+<instance part="C5" gate="G$1" x="111.76" y="213.36"/>
 </instances>
 <busses>
@@
 <wire x1="43.18" y1="226.06" x2="43.18" y2="220.98" width="0.1524" layer="91"/>
 </segment>
-<segment>
-<pinref part="P+1" gate="1" pin="+5V"/>
-<pinref part="PAD3" gate="P" pin="P"/>
-<wire x1="160.02" y1="226.06" x2="160.02" y2="220.98" width="0.1524" layer="91"/>
-</segment>
-</net>
-<net name="+3V3" class="0">
-<segment>
-<pinref part="IC1" gate="G$1" pin="VOUT"/>
-<pinref part="C3" gate="G$1" pin="+"/>
-<wire x1="93.98" y1="218.44" x2="99.06" y2="218.44" width="0.1524" layer="91"/>
-<wire x1="99.06" y1="218.44" x2="99.06" y2="215.9" width="0.1524" layer="91"/>
-<pinref part="+3V2" gate="G$1" pin="+3V3"/>
-<wire x1="99.06" y1="226.06" x2="99.06" y2="218.44" width="0.1524" layer="91"/>
-<pinref part="R1" gate="G$1" pin="2"/>
-<wire x1="99.06" y1="218.44" x2="104.14" y2="218.44" width="0.1524" layer="91"/>
-<junction x="99.06" y="218.44"/>
-</segment>
-<segment>
-<pinref part="+3V1" gate="G$1" pin="+3V3"/>
-<pinref part="C1" gate="G$1" pin="+"/>
-<wire x1="50.8" y1="152.4" x2="50.8" y2="149.86" width="0.1524" layer="91"/>
-<pinref part="SV1" gate="G$1" pin="12"/>
-<wire x1="50.8" y1="149.86" x2="50.8" y2="147.32" width="0.1524" layer="91"/>
-<wire x1="60.96" y1="154.94" x2="55.88" y2="154.94" width="0.1524" layer="91"/>
-<wire x1="55.88" y1="154.94" x2="55.88" y2="149.86" width="0.1524" layer="91"/>
-<wire x1="55.88" y1="149.86" x2="50.8" y2="149.86" width="0.1524" layer="91"/>
-<junction x="50.8" y="149.86"/>
-</segment>
-<segment>
-<pinref part="+3V3" gate="G$1" pin="+3V3"/>
-<wire x1="71.12" y1="142.24" x2="71.12" y2="139.7" width="0.1524" layer="91"/>
-<pinref part="SV2" gate="1" pin="1"/>
-<wire x1="71.12" y1="139.7" x2="76.2" y2="139.7" width="0.1524" layer="91"/>
-<wire x1="76.2" y1="139.7" x2="76.2" y2="147.32" width="0.1524" layer="91"/>
-</segment>
 </net>
 <net name="GND" class="0">
@@
 <pinref part="C3" gate="G$1" pin="-"/>
 <pinref part="SUPPLY7" gate="GND" pin="GND"/>
-<wire x1="99.06" y1="208.28" x2="99.06" y2="203.2" width="0.1524" layer="91"/>
+<wire x1="96.52" y1="208.28" x2="96.52" y2="203.2" width="0.1524" layer="91"/>
 </segment>
 <segment>
@@
 </segment>
 <segment>
-<pinref part="C4" gate="G$1" pin="-"/>
 <pinref part="SUPPLY9" gate="GND" pin="GND"/>
-<wire x1="116.84" y1="208.28" x2="116.84" y2="203.2" width="0.1524" layer="91"/>
+<wire x1="111.76" y1="208.28" x2="111.76" y2="203.2" width="0.1524" layer="91"/>
+<pinref part="C5" gate="G$1" pin="2"/>
 </segment>
 <segment>
@@
 <pinref part="C1" gate="G$1" pin="-"/>
 <pinref part="SUPPLY3" gate="GND" pin="GND"/>
-<wire x1="50.8" y1="139.7" x2="50.8" y2="137.16" width="0.1524" layer="91"/>
+<wire x1="50.8" y1="137.16" x2="50.8" y2="134.62" width="0.1524" layer="91"/>
 </segment>
 </net>
@@
 <segment>
 <pinref part="R1" gate="G$1" pin="1"/>
-<pinref part="C4" gate="G$1" pin="+"/>
-<wire x1="114.3" y1="218.44" x2="116.84" y2="218.44" width="0.1524" layer="91"/>
-<wire x1="116.84" y1="218.44" x2="116.84" y2="215.9" width="0.1524" layer="91"/>
-<label x="137.16" y="218.44" size="1.27" layer="95" xref="yes"/>
-<wire x1="116.84" y1="218.44" x2="137.16" y2="218.44" width="0.1524" layer="91"/>
-<junction x="116.84" y="218.44"/>
+<wire x1="109.22" y1="218.44" x2="111.76" y2="218.44" width="0.1524" layer="91"/>
+<wire x1="111.76" y1="218.44" x2="111.76" y2="215.9" width="0.1524" layer="91"/>
+<label x="132.08" y="218.44" size="1.27" layer="95" xref="yes"/>
+<wire x1="111.76" y1="218.44" x2="132.08" y2="218.44" width="0.1524" layer="91"/>
+<junction x="111.76" y="218.44"/>
+<pinref part="C5" gate="G$1" pin="1"/>
 </segment>
 <segment>
@@
 </segment>
 </net>
+<net name="VCC" class="0">
+<segment>
+<pinref part="IC1" gate="G$1" pin="VOUT"/>
+<pinref part="C3" gate="G$1" pin="+"/>
+<wire x1="93.98" y1="218.44" x2="96.52" y2="218.44" width="0.1524" layer="91"/>
+<wire x1="96.52" y1="218.44" x2="96.52" y2="215.9" width="0.1524" layer="91"/>
+<wire x1="96.52" y1="226.06" x2="96.52" y2="218.44" width="0.1524" layer="91"/>
+<pinref part="R1" gate="G$1" pin="2"/>
+<wire x1="96.52" y1="218.44" x2="99.06" y2="218.44" width="0.1524" layer="91"/>
+<junction x="96.52" y="218.44"/>
+<pinref part="SUPPLY4" gate="G$1" pin="VCC"/>
+</segment>
+<segment>
+<pinref part="PAD3" gate="P" pin="P"/>
+<wire x1="160.02" y1="226.06" x2="160.02" y2="220.98" width="0.1524" layer="91"/>
+<pinref part="SUPPLY13" gate="G$1" pin="VCC"/>
+</segment>
+<segment>
+<pinref part="C1" gate="G$1" pin="+"/>
+<wire x1="50.8" y1="149.86" x2="50.8" y2="147.32" width="0.1524" layer="91"/>
+<pinref part="SV1" gate="G$1" pin="12"/>
+<wire x1="50.8" y1="147.32" x2="50.8" y2="144.78" width="0.1524" layer="91"/>
+<wire x1="60.96" y1="154.94" x2="55.88" y2="154.94" width="0.1524" layer="91"/>
+<wire x1="55.88" y1="154.94" x2="55.88" y2="147.32" width="0.1524" layer="91"/>
+<wire x1="55.88" y1="147.32" x2="50.8" y2="147.32" width="0.1524" layer="91"/>
+<junction x="50.8" y="147.32"/>
+<pinref part="SUPPLY14" gate="G$1" pin="VCC"/>
+</segment>
+<segment>
+<wire x1="71.12" y1="139.7" x2="71.12" y2="137.16" width="0.1524" layer="91"/>
+<pinref part="SV2" gate="1" pin="1"/>
+<wire x1="71.12" y1="137.16" x2="76.2" y2="137.16" width="0.1524" layer="91"/>
+<wire x1="76.2" y1="137.16" x2="76.2" y2="147.32" width="0.1524" layer="91"/>
+<pinref part="SUPPLY15" gate="G$1" pin="VCC"/>
+</segment>
+</net>

Commit message: 1st completion
1st completion
Parts:
- removed C5: 10uF, rcl:C-USC1206
- added C4: 10uF, rcl:C-USC1206
- added F1: (no value), fuse:GSH15
- added PAD4, PAD5, PAD6: (no value), wirepad:2,54/0,8
- added PAD7: +5V, wirepad:2,54/0,8
- added PAD8: GND, wirepad:2,54/0,8
- added PAD9: +3.3V, wirepad:2,54/0,8
- added SV4: (no value), con-lstb:MA03-1
- added X1: 5202-03-N-02, con-ebyelectro:5202-03-N-02
- PAD1: value +5V -> AC-; device wirepad:2,54/0,8 -> wirepad:2,54/1,0
- PAD2: value GND -> AC+; device wirepad:2,54/0,8 -> wirepad:2,54/1,0
- PAD3: value +3.3V -> (none)
Connections:
- new net AC+: X1-3.1
- new net LAMP: X1-2.1
- new net N$1: PAD1.P, PAD3.P
- new net N$2: F1.1, PAD2.P
- new net N$3: F1.2, PAD4.P
- net +5V: now also PAD5.P, PAD7.P, SV4.1; no longer PAD1.P
- net /RESET: now also C4.1; no longer C5.1
- net GND: now also C4.2, PAD6.P, PAD8.P, SV4.2; no longer C5.2, PAD2.P
- net PC6/MODE/DIO0: now also SV4.3
- net VCC: now also PAD9.P; no longer PAD3.P
Other:
- note added: "AC"
- note added: "MSC0405"
- note added: "Relay Board"
- moved on the sheet: C2, C3, IC1, PAD1, PAD2, PAD3, R1, SV2

Commit message: Merge to Schematics
Parts:
- added C5: 4.7uF, rcl:CPOL-USSANYO_SMD_A5
- added SV5, SV6: (no value), con-lstb:MA13-1
- added SV7: (no value), con-lstb:MA08-1
- added SV8, SV9: (no value), con-lstb:MA12-1
Connections:
- removed net PB1/TXD: SV3.6
- removed net PB2/RXD: SV3.5
- new net A0: SV9.5
- new net A1: SV9.6
- new net A2: SV9.7
- new net A3: SV9.8
- new net D10: SV9.1
- new net D2: SV8.8
- new net D3: SV8.7
- new net D4: SV8.6
- new net D5: SV8.5
- new net D6: SV8.4
- new net D7: SV8.3
- new net D8: SV8.2
- new net D9: SV8.1
- new net GND1: SV6.1, SV6.13
- new net MISO: SV9.3
- new net MOSI: SV9.2
- new net RAW: SV9.12
- new net RESET: SV8.10, SV9.10
- new net RXD: SV3.5, SV5.1
- new net RXI: SV8.11
- new net SCK: SV9.4
- new net TXD: SV3.6, SV5.2
- new net TXO: SV8.12
- net +5V: now also SV9.9
- net GND: now also C5.-, SV5.13, SV8.9, SV9.11
- net PA3/NSSEL/DIO8: now also SV4.3
- net PC6/MODE/DIO0: no longer SV4.3
- net VCC: now also C5.+, SV5.12
Other:
- note added: "Arduino Pro Mini"
- note added: "HC-06"
- note added: "RX"
- note added: "TX"
- note added: "ZigBee"
- moved on the sheet: SV4, X1-1, X1-2, X1-3
