File: ZigBeeHA/main.brd (EAGLE design)
At the start: 100 x 80 mm, 34 parts, among them IC1 REG1117, Q1 2N3904, X1 5202-03-N-02

Commit message: RPi version updated
Parts:
- removed C2: 10uF, rcl:SANYO-OSCON_SMD_A5
- removed C3: 4.7uF, rcl:SANYO-OSCON_SMD_A5
- removed C4: 10uF, rcl:C1206
- removed F1: (no value), fuse:GSH15
- removed IC1: REG1117, burr-brown:SOT223
- removed PAD1: AC-, wirepad:2,54/1,0
- removed PAD2: AC+, wirepad:2,54/1,0
- removed PAD3, PAD4, PAD5, PAD6: (no value), wirepad:2,54/0,8
- removed PAD7: +5V, wirepad:2,54/0,8
- removed PAD8: GND, wirepad:2,54/0,8
- removed PAD9: +3.3V, wirepad:2,54/0,8
- removed R1: 10K, rcl:M1206
- removed SV4: (no value), con-lstb:MA03-1
- removed X1: 5202-03-N-02, con-ebyelectro:5202-03-N-02
Connections:
- removed net AC+: X1.3
- removed net LAMP: X1.2
- removed net N$1: PAD1.1, PAD3.1
- removed net N$2: F1.1, PAD2.1
- removed net N$3: F1.2, PAD4.1
- net +5V: no longer C2.+, IC1.3, PAD5.1, PAD7.1, SV4.1
- net /RESET: no longer C4.1, R1.1
- net GND: no longer C2.-, C3.-, C4.2, IC1.1, PAD6.1, PAD8.1, SV4.2
- net PA3/NSSEL/DIO8: no longer SV4.3
- net VCC: no longer C3.+, IC1.2, PAD9.1, R1.2
Routing:
- net VCC: track 1.39 -> 0.00 mm
- net GND: track 1.19 -> 0.00 mm
