File: Devention/devention.sch (EAGLE design)
At the start: 33 parts, among them Q4 #MHz, U1 ATMEGA328L, U2 ###V, U3 HC_05

Commit message: update devention
Connections:
- net BT_RXD: now also U3.RX
- net BT_TXD: now also U3.TX
Changed lines of the file:
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@@
 <?xml version="1.0" encoding="utf-8"?>
 <!DOCTYPE eagle SYSTEM "eagle.dtd">
-<eagle version="6.5.0">
+<eagle version="7.2.0">
 <drawing>
 <settings>
@@
 <label x="137.16" y="119.38" size="1.27" layer="95" xref="yes"/>
 </segment>
+<segment>
+<pinref part="U3" gate="G$1" pin="TX"/>
+<wire x1="170.18" y1="58.42" x2="152.4" y2="58.42" width="0.1524" layer="91"/>
+<label x="152.4" y="58.42" size="1.27" layer="95" xref="yes"/>
+</segment>
 </net>
 <net name="BT_RXD" class="0">
@@
 <label x="146.304" y="116.84" size="1.27" layer="95" rot="R180" xref="yes"/>
 </segment>
-</net>
+<segment>
+<pinref part="U3" gate="G$1" pin="RX"/>
+<wire x1="170.18" y1="55.88" x2="162.56" y2="55.88" width="0.1524" layer="91"/>
+<label x="162.56" y="55.88" size="1.27" layer="95" rot="MR0" xref="yes"/>
+</segment>
+</net>
