File: Deviation/deviation.sch (EAGLE design)
At the start: 33 parts, among them Q4 #MHz, U1 ATMEGA328L, U2 ###V, U3 HC_05

Commit message: -- Folder name changed to Deviation --
micro USB male connector added to schematic
Parts:
- added J1: MICRO_USB_B_MALE_HIROSE_ZX80-B-5S, connector:MICRO_USB_B_MALE_HIROSE_ZX80-B-5S
- Q4: value #MHz -> 8MHz
Connections:
- net GND: now also J1.GND, J1.ID
- net RAW: now also J1.+5V
Other:
- moved on the sheet: C10, C13, C19, LED1, R16, U2
Changed lines of the file:
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@@
 <part name="P+11" library="SparkFun" deviceset="3.3V" device="" value="VCC"/>
 <part name="P+15" library="SparkFun" deviceset="3.3V" device="" value="VCC"/>
-<part name="Q4" library="SparkFun" deviceset="RESONATOR" device="SMD" value="#MHz"/>
+<part name="Q4" library="SparkFun" deviceset="RESONATOR" device="SMD" value="8MHz"/>
 <part name="GND4" library="SparkFun" deviceset="GND" device=""/>
 <part name="U1" library="SparkFun" deviceset="ATMEGA168" device="" value="ATMEGA328L"/>
@@
 <part name="R17" library="SparkFun" deviceset="RESISTOR" device="0402" value="180"/>
 <part name="SUPPLY1" library="supply2" deviceset="GND" device=""/>
+<part name="J1" library="connector" deviceset="MICRO_USB_B_MALE_HIROSE_ZX80-B-5S" device=""/>
+<part name="GND1" library="SparkFun" deviceset="GND" device=""/>
 </parts>
 <sheets>
@@
 <attribute name="VALUE" x="130.048" y="116.84" size="1.778" layer="96"/>
 </instance>
-<instance part="C10" gate="G$1" x="60.96" y="48.26"/>
-<instance part="C13" gate="G$1" x="53.34" y="50.8"/>
-<instance part="GND25" gate="1" x="53.34" y="40.64"/>
-<instance part="GND26" gate="1" x="60.96" y="40.64"/>
-<instance part="R16" gate="G$1" x="73.66" y="48.26" rot="R90"/>
-<instance part="LED1" gate="G$1" x="73.66" y="38.1"/>
-<instance part="GND28" gate="1" x="73.66" y="27.94"/>
-<instance part="U2" gate="G$1" x="40.64" y="50.8"/>
-<instance part="C19" gate="G$1" x="17.78" y="48.26"/>
-<instance part="GND30" gate="1" x="25.4" y="38.1"/>
-<instance part="GND32" gate="1" x="17.78" y="38.1"/>
-<instance part="P+12" gate="G$1" x="73.66" y="58.42"/>
+<instance part="C10" gate="G$1" x="106.68" y="43.18"/>
+<instance part="C13" gate="G$1" x="99.06" y="45.72"/>
+<instance part="GND25" gate="1" x="99.06" y="35.56"/>
+<instance part="GND26" gate="1" x="106.68" y="35.56"/>
+<instance part="R16" gate="G$1" x="119.38" y="43.18" rot="R90"/>
+<instance part="LED1" gate="G$1" x="119.38" y="33.02"/>
+<instance part="GND28" gate="1" x="119.38" y="22.86"/>
+<instance part="U2" gate="G$1" x="86.36" y="45.72"/>
+<instance part="C19" gate="G$1" x="63.5" y="43.18"/>
+<instance part="GND30" gate="1" x="71.12" y="33.02"/>
+<instance part="GND32" gate="1" x="63.5" y="33.02"/>
+<instance part="P+12" gate="G$1" x="119.38" y="53.34"/>
 <instance part="SUPPLY12" gate="GND" x="165.1" y="5.08"/>
 <instance part="C5" gate="G$1" x="157.48" y="15.24"/>
@@
 <instance part="R17" gate="G$1" x="238.76" y="33.02"/>
 <instance part="SUPPLY1" gate="GND" x="246.38" y="27.94"/>
+<instance part="J1" gate="G$1" x="30.48" y="45.72" rot="MR0"/>
+<instance part="GND1" gate="1" x="45.72" y="33.02"/>
 </instances>
 <busses>
@@
 </segment>
 <segment>
-<wire x1="48.26" y1="55.88" x2="53.34" y2="55.88" width="0.1524" layer="91"/>
-<wire x1="53.34" y1="55.88" x2="60.96" y2="55.88" width="0.1524" layer="91"/>
-<wire x1="60.96" y1="55.88" x2="73.66" y2="55.88" width="0.1524" layer="91"/>
-<wire x1="73.66" y1="55.88" x2="73.66" y2="58.42" width="0.1524" layer="91"/>
-<wire x1="73.66" y1="55.88" x2="73.66" y2="53.34" width="0.1524" layer="91"/>
-<wire x1="60.96" y1="55.88" x2="60.96" y2="53.34" width="0.1524" layer="91"/>
-<wire x1="53.34" y1="55.88" x2="53.34" y2="53.34" width="0.1524" layer="91"/>
-<junction x="73.66" y="55.88"/>
-<junction x="60.96" y="55.88"/>
-<junction x="53.34" y="55.88"/>
+<wire x1="93.98" y1="50.8" x2="99.06" y2="50.8" width="0.1524" layer="91"/>
+<wire x1="99.06" y1="50.8" x2="106.68" y2="50.8" width="0.1524" layer="91"/>
+<wire x1="106.68" y1="50.8" x2="119.38" y2="50.8" width="0.1524" layer="91"/>
+<wire x1="119.38" y1="50.8" x2="119.38" y2="53.34" width="0.1524" layer="91"/>
+<wire x1="119.38" y1="50.8" x2="119.38" y2="48.26" width="0.1524" layer="91"/>
+<wire x1="106.68" y1="50.8" x2="106.68" y2="48.26" width="0.1524" layer="91"/>
+<wire x1="99.06" y1="50.8" x2="99.06" y2="48.26" width="0.1524" layer="91"/>
+<junction x="119.38" y="50.8"/>
+<junction x="106.68" y="50.8"/>
+<junction x="99.06" y="50.8"/>
 <pinref part="U2" gate="G$1" pin="OUT"/>
 <pinref part="P+12" gate="G$1" pin="3.3V"/>
@@
 </segment>
 <segment>
-<wire x1="53.34" y1="43.18" x2="53.34" y2="45.72" width="0.1524" layer="91"/>
+<wire x1="99.06" y1="38.1" x2="99.06" y2="40.64" width="0.1524" layer="91"/>
 <pinref part="C13" gate="G$1" pin="-"/>
 <pinref part="GND25" gate="1" pin="GND"/>
 </segment>
 <segment>
-<wire x1="60.96" y1="43.18" x2="60.96" y2="45.72" width="0.1524" layer="91"/>
+<wire x1="106.68" y1="38.1" x2="106.68" y2="40.64" width="0.1524" layer="91"/>
 <pinref part="C10" gate="G$1" pin="2"/>
 <pinref part="GND26" gate="1" pin="GND"/>
 </segment>
 <segment>
-<wire x1="73.66" y1="30.48" x2="73.66" y2="33.02" width="0.1524" layer="91"/>
+<wire x1="119.38" y1="25.4" x2="119.38" y2="27.94" width="0.1524" layer="91"/>
 <pinref part="LED1" gate="G$1" pin="C"/>
 <pinref part="GND28" gate="1" pin="GND"/>
 </segment>
 <segment>
-<wire x1="30.48" y1="50.8" x2="25.4" y2="50.8" width="0.1524" layer="91"/>
-<wire x1="25.4" y1="50.8" x2="25.4" y2="40.64" width="0.1524" layer="91"/>
+<wire x1="76.2" y1="45.72" x2="71.12" y2="45.72" width="0.1524" layer="91"/>
+<wire x1="71.12" y1="45.72" x2="71.12" y2="35.56" width="0.1524" layer="91"/>
 <pinref part="U2" gate="G$1" pin="GND"/>
 <pinref part="GND30" gate="1" pin="GND"/>
 </segment>
 <segment>
-<wire x1="17.78" y1="40.64" x2="17.78" y2="43.18" width="0.1524" layer="91"/>
+<wire x1="63.5" y1="35.56" x2="63.5" y2="38.1" width="0.1524" layer="91"/>
 <pinref part="C19" gate="G$1" pin="-"/>
 <pinref part="GND32" gate="1" pin="GND"/>
@@
 <wire x1="243.84" y1="33.02" x2="246.38" y2="33.02" width="0.1524" layer="91"/>
 <wire x1="246.38" y1="33.02" x2="246.38" y2="30.48" width="0.1524" layer="91"/>
+</segment>
+<segment>
+<pinref part="J1" gate="G$1" pin="GND"/>
+<wire x1="38.1" y1="40.64" x2="45.72" y2="40.64" width="0.1524" layer="91"/>
+<wire x1="45.72" y1="40.64" x2="45.72" y2="35.56" width="0.1524" layer="91"/>
+<pinref part="GND1" gate="1" pin="GND"/>
+<pinref part="J1" gate="G$1" pin="ID"/>
+<wire x1="38.1" y1="43.18" x2="45.72" y2="43.18" width="0.1524" layer="91"/>
+<wire x1="45.72" y1="43.18" x2="45.72" y2="40.64" width="0.1524" layer="91"/>
+<junction x="45.72" y="40.64"/>
 </segment>
 </net>
@@
 <net name="N$38" class="0">
 <segment>
-<wire x1="73.66" y1="40.64" x2="73.66" y2="43.18" width="0.1524" layer="91"/>
+<wire x1="119.38" y1="35.56" x2="119.38" y2="38.1" width="0.1524" layer="91"/>
 <pinref part="R16" gate="G$1" pin="1"/>
 <pinref part="LED1" gate="G$1" pin="A"/>
@@
 <net name="RAW" class="1">
 <segment>
-<wire x1="27.94" y1="55.88" x2="30.48" y2="55.88" width="0.1524" layer="91"/>
-<wire x1="30.48" y1="45.72" x2="27.94" y2="45.72" width="0.1524" layer="91"/>
-<wire x1="27.94" y1="45.72" x2="27.94" y2="55.88" width="0.1524" layer="91"/>
-<wire x1="17.78" y1="55.88" x2="27.94" y2="55.88" width="0.1524" layer="91"/>
-<wire x1="17.78" y1="50.8" x2="17.78" y2="55.88" width="0.1524" layer="91"/>
-<wire x1="17.78" y1="55.88" x2="10.16" y2="55.88" width="0.1524" layer="91"/>
-<junction x="27.94" y="55.88"/>
-<junction x="17.78" y="55.88"/>
-<label x="10.16" y="55.88" size="1.778" layer="95"/>
+<wire x1="73.66" y1="50.8" x2="76.2" y2="50.8" width="0.1524" layer="91"/>
+<wire x1="76.2" y1="40.64" x2="73.66" y2="40.64" width="0.1524" layer="91"/>
+<wire x1="73.66" y1="40.64" x2="73.66" y2="50.8" width="0.1524" layer="91"/>
+<wire x1="63.5" y1="50.8" x2="73.66" y2="50.8" width="0.1524" layer="91"/>
+<wire x1="63.5" y1="45.72" x2="63.5" y2="50.8" width="0.1524" layer="91"/>
+<junction x="73.66" y="50.8"/>
+<junction x="63.5" y="50.8"/>
+<label x="55.88" y="50.8" size="1.778" layer="95"/>
 <pinref part="U2" gate="G$1" pin="IN"/>
 <pinref part="U2" gate="G$1" pin="EN"/>
 <pinref part="C19" gate="G$1" pin="+"/>
-</segment>
-</net>
+<pinref part="J1" gate="G$1" pin="+5V"/>
+<wire x1="38.1" y1="50.8" x2="63.5" y2="50.8" width="0.1524" layer="91"/>
+</segment>
+</net>
